Commit message: added 4 cnt points per leg

File: build/lib/robot_properties_talos/robot_properties_talos/urdf/talos.urdf (robot description, URDF)
Before this commit: robot talos, 62 links, 61 joints
Links:
- added link left_sole_link3, mass 0.01
- added link left_sole_link4, mass 0.01
- added link right_sole_link3, mass 0.01
- added link right_sole_link4, mass 0.01
Joints:
- added joint leg_left_sole3_fix_joint: type fixed, parent leg_left_6_link, child left_sole_link3, origin xyz=-0.10 0.05 -0.107 rpy=0 0 0, axis 1 0 0
- added joint leg_left_sole4_fix_joint: type fixed, parent leg_left_6_link, child left_sole_link4, origin xyz=0.12 0.05 -0.107 rpy=0 0 0, axis 1 0 0
- added joint leg_right_sole3_fix_joint: type fixed, parent leg_right_6_link, child right_sole_link3, origin xyz=-0.10 0.05 -0.107 rpy=0 0 0, axis 1 0 0
- added joint leg_right_sole4_fix_joint: type fixed, parent leg_right_6_link, child right_sole_link4, origin xyz=0.12 0.05 -0.107 rpy=0 0 0, axis 1 0 0
- joint gripper_left_fingertip_1_joint: type revolute -> fixed
- joint gripper_left_fingertip_2_joint: type revolute -> fixed
- joint gripper_left_fingertip_3_joint: type revolute -> fixed
- joint gripper_left_inner_double_joint: type revolute -> fixed
- joint gripper_left_inner_single_joint: type revolute -> fixed
- joint gripper_left_joint: type revolute -> fixed
- joint gripper_left_motor_single_joint: type revolute -> fixed
- joint gripper_right_fingertip_1_joint: type revolute -> fixed
- joint gripper_right_fingertip_2_joint: type revolute -> fixed
- joint gripper_right_fingertip_3_joint: type revolute -> fixed
- joint gripper_right_inner_double_joint: type revolute -> fixed
- joint gripper_right_inner_single_joint: type revolute -> fixed
- joint gripper_right_joint: type revolute -> fixed
- joint gripper_right_motor_single_joint: type revolute -> fixed
- joint head_1_joint: type revolute -> fixed
- joint head_2_joint: type revolute -> fixed
- joint leg_left_sole1_fix_joint: origin xyz=-0.10 0.00 -0.107 rpy=0 0 0 -> xyz=-0.10 -0.05 -0.107 rpy=0 0 0
- joint leg_left_sole2_fix_joint: origin xyz=0.12 0.00 -0.107 rpy=0 0 0 -> xyz=0.12 -0.05 -0.107 rpy=0 0 0
- joint leg_right_sole1_fix_joint: origin xyz=-0.10 0.00 -0.107 rpy=0 0 0 -> xyz=-0.10 -0.05 -0.107 rpy=0 0 0
- joint leg_right_sole2_fix_joint: origin xyz=0.12 0.00 -0.107 rpy=0 0 0 -> xyz=0.12 -.05 -0.107 rpy=0 0 0
